Commit message: second big commit (reorder the files paths, implementing properly SLAM, modifying TFs links, correct cmake, add options to activate or no Rviz or gazebo headless, etc...)

File: models/simple_robot/test/urdf/test.urdf (robot description, URDF)
Before this commit: robot test, 2 links, 1 joints
Links:
- link base_link: geometry collision mesh filename=file:///workspaces/mam_eurobot_2026/models/simple_robot/tes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; visual mesh filename=file:///workspaces/mam_eurobot_2026/models/simple_robot/tes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
- link servo: geometry collision mesh filename=file:///workspaces/mam_eurobot_2026/models/simple_robot/tes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; visual mesh filename=file:///workspaces/mam_eurobot_2026/models/simple_robot/tes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
